File: light-tone-pedal.sch (KiCad schematic (older format))
At the start: 22 parts, among them U1 LM358AP

Commit message: Added pwr_flag symbol to schematic in eeschema.
Parts:
- C1, C2, C3: footprint (none) -> Capacitors_THT:C_Disc_D7.0mm_W2.5mm_P5.00mm
- C_HIGH1: footprint (none) -> Capacitors_THT:C_Rect_L24.0mm_W7.0mm_P22.50mm_MKT
- C_LOW1: footprint (none) -> Capacitors_THT:C_Rect_L13.0mm_W8.0mm_P10.00mm_FKS3_FKP3_MKS4
- R1, R2, R_HIGH1, R_LDR1, R_LDRLOW1, R_LOW1: footprint (none) -> Resistors_THT:R_Axial_DIN0207_L6.3mm_D2.5mm_P7.62mm_Horizontal
- U1: footprint DIP254P762X508-8 -> (none)
Changed lines of the file:
@@
 F 0 "R_LDRLOW1" V 5500 3150 50  0000 C CNN
 F 1 "3k" V 5586 3150 50  0000 C CNN
-F 2 "" H 5700 3150 50  0001 C CNN
+F 2 "Resistors_THT:R_Axial_DIN0207_L6.3mm_D2.5mm_P7.62mm_Horizontal" H 5700 3150 50  0001 C CNN
 F 3 "~" H 5700 3150 50  0001 C CNN
 	1    5700 3150
@@
 F 0 "R_LOW1" V 5800 3400 50  0000 C CNN
 F 1 "24k" V 5900 3400 50  0000 C CNN
-F 2 "" H 5700 3400 50  0001 C CNN
+F 2 "Resistors_THT:R_Axial_DIN0207_L6.3mm_D2.5mm_P7.62mm_Horizontal" H 5700 3400 50  0001 C CNN
 F 3 "~" H 5700 3400 50  0001 C CNN
 	1    5700 3400
@@
 F 0 "C_LOW1" H 6528 3696 50  0000 L CNN
 F 1 "0.022u" H 6528 3605 50  0000 L CNN
-F 2 "" H 6350 3650 50  0001 C CNN
+F 2 "Capacitors_THT:C_Rect_L13.0mm_W8.0mm_P10.00mm_FKS3_FKP3_MKS4" H 6350 3650 50  0001 C CNN
 F 3 "~" H 6350 3650 50  0001 C CNN
 	1    6350 3650
@@
 F 0 "R_LDR1" H 6668 1696 50  0000 L CNN
 F 1 "11k" H 6668 1605 50  0000 L CNN
-F 2 "" H 6600 1650 50  0001 C CNN
+F 2 "Resistors_THT:R_Axial_DIN0207_L6.3mm_D2.5mm_P7.62mm_Horizontal" H 6600 1650 50  0001 C CNN
 F 3 "~" H 6600 1650 50  0001 C CNN
 	1    6600 1650
@@
 F 0 "R_HIGH1" H 5850 1750 50  0000 L CNN
 F 1 "24k" H 5950 1650 50  0000 L CNN
-F 2 "" H 6200 1650 50  0001 C CNN
+F 2 "Resistors_THT:R_Axial_DIN0207_L6.3mm_D2.5mm_P7.62mm_Horizontal" H 6200 1650 50  0001 C CNN
 F 3 "~" H 6200 1650 50  0001 C CNN
 	1    6200 1650
@@
 F 0 "C_HIGH1" V 5385 2150 50  0000 C CNN
 F 1 "5600p" V 5476 2150 50  0000 C CNN
-F 2 "" H 5700 2150 50  0001 C CNN
+F 2 "Capacitors_THT:C_Rect_L24.0mm_W7.0mm_P22.50mm_MKT" H 5700 2150 50  0001 C CNN
 F 3 "~" H 5700 2150 50  0001 C CNN
 	1    5700 2150
@@
 F 0 "C2" V 7335 2750 50  0000 C CNN
 F 1 "1u" V 7426 2750 50  0000 C CNN
-F 2 "" H 7650 2750 50  0001 C CNN
+F 2 "Capacitors_THT:C_Disc_D7.0mm_W2.5mm_P5.00mm" H 7650 2750 50  0001 C CNN
 F 3 "~" H 7650 2750 50  0001 C CNN
 	1    7650 2750
@@
 F 0 "U1" H 6150 5720 50  0000 C CNN
 F 1 "LM358AP" H 6150 5629 50  0000 C CNN
-F 2 "DIP254P762X508-8" H 6150 5150 50  0001 L BNN
+F 2 "" H 6150 5150 50  0001 L BNN
 F 3 "" H 6150 5150 50  0001 L BNN
 F 4 "LM358AP" H 6150 5150 50  0001 L BNN "Field4"
@@
 Wire Wire Line
 	7300 4300 4750 4300
-Wire Wire Line
-	4750 4300 4750 2650
 Connection ~ 7300 4950
 Wire Wire Line
@@
 F 0 "R2" H 7168 5346 50  0000 L CNN
 F 1 "100k" H 7168 5255 50  0000 L CNN
-F 2 "" H 7100 5300 50  0001 C CNN
+F 2 "Resistors_THT:R_Axial_DIN0207_L6.3mm_D2.5mm_P7.62mm_Horizontal" H 7100 5300 50  0001 C CNN
 F 3 "~" H 7100 5300 50  0001 C CNN
 	1    7100 5300
@@
 F 0 "R1" H 4918 5746 50  0000 L CNN
 F 1 "1k" H 4918 5655 50  0000 L CNN
-F 2 "" H 4850 5700 50  0001 C CNN
+F 2 "Resistors_THT:R_Axial_DIN0207_L6.3mm_D2.5mm_P7.62mm_Horizontal" H 4850 5700 50  0001 C CNN
 F 3 "~" H 4850 5700 50  0001 C CNN
 	1    4850 5700
@@
 F 0 "C1" H 5028 6346 50  0000 L CNN
 F 1 "0.1u" H 5028 6255 50  0000 L CNN
-F 2 "" H 4850 6300 50  0001 C CNN
+F 2 "Capacitors_THT:C_Disc_D7.0mm_W2.5mm_P5.00mm" H 4850 6300 50  0001 C CNN
 F 3 "~" H 4850 6300 50  0001 C CNN
 	1    4850 6300
@@
 F 0 "C3" V 8115 4050 50  0000 C CNN
 F 1 "1u" V 8024 4050 50  0000 C CNN
-F 2 "" H 7800 4050 50  0001 C CNN
+F 2 "Capacitors_THT:C_Disc_D7.0mm_W2.5mm_P5.00mm" H 7800 4050 50  0001 C CNN
 F 3 "~" H 7800 4050 50  0001 C CNN
 	1    7800 4050
@@
 Wire Wire Line
 	8250 4600 8250 4550
+Wire Wire Line
+	4750 4300 4750 2650
 $EndSCHEMATC
