File: light-tone-pedal.sch (KiCad schematic (older format))
At the start: 48 parts, among them U1 LM358AP, U2 LM358AP, U3 LM358AP

Commit message: I removed the low-pass filter since it was not working out too well in pcb design.
Parts:
- removed Cpow1: 100u, Capacitor_THT:C_Disc_D7.0mm_W2.5mm_P5.00mm, symbol PSPICE:CAP
- removed Rpow1: 200, Resistor_THT:R_Axial_DIN0207_L6.3mm_D2.5mm_P7.62mm_Horizontal, symbol PSPICE:R
- C1, C10, C2, C3, C4, C5, C6, C7, C8, C9: symbol PSPICE:CAP -> light-tone-pedal-rescue:CAP-PSPICE
- D1, D2: symbol Diode:CQY99 -> light-tone-pedal-rescue:CQY99-Diode
- LDR1, LDR2, R1, R10, R11, R13, R14, R15, R16, R17, R18, R2, R3, R4, R5, R6, R7, R8, RPOT1, RPOT10, RPOT2, RPOT3, RPOT4, RPOT5, RPOT6, RPOT7, RPOT8, RPOT9: symbol PSPICE:R -> light-tone-pedal-rescue:R-PSPICE
- U1, U2, U3: symbol LM358AP:LM358AP -> light-tone-pedal-rescue:LM358AP-LM358AP
- V1: symbol PSPICE:VSOURCE -> light-tone-pedal-rescue:VSOURCE-PSPICE
Connections:
- net vcc_filtered is gone; now on net VCC: R15.1, R3.1, U1.8 (VCC), U2.8 (VCC), U3.8 (VCC)
